File: shield.kicad_sch (KiCad schematic)
At the start: 10 parts, among them J1 DEVKIT_C2000_ROW_A, J10 ESP32_C6_DEVKITC_1_J3, J2 DEVKIT_C2000_ROW_B, J3 NAPPE_ADC1, J4 NAPPE_ADC2, J5 NAPPE_PWM, J6 NAPPE_GPIO, J7 ALIM_5V, J8 ALIM_5V, J9 ESP32_C6_DEVKITC_1_J1

Commit message: Separation connecteurs/protection en sous-feuilles, correction annotation, assignation des empreintes
Eclate shield.kicad_sch en sous-feuilles (connecteurs devkit, nappes, DC,
chaines de protection BAT54S) et corrige la duplication de reference J1
entre DEVKIT_C2000_ROW_A et le connecteur d'alimentation de dc.kicad_sch.
Assigne une empreinte a tous les composants places (R/C en 0805, BAT54S en
SOT-23, cavaliers/connecteurs 2 broches en PinHeader 1x02, zener de
protection en SMC) et cree l'empreinte custom NCM3S1205MC d'apres le
datasheet Murata pour debloquer la mise a jour du PCB depuis le schema.

Co-Authored-By: Claude Sonnet 5 <noreply@anthropic.com>
Parts:
- removed J1: DEVKIT_C2000_ROW_A, symbol C2000_Devkit_Connectors:DEVKIT_C2000_ROW_A
- removed J10: ESP32_C6_DEVKITC_1_J3, symbol ESP32_C6_Devkit:ESP32_C6_DEVKITC_1_J3
- removed J2: DEVKIT_C2000_ROW_B, symbol C2000_Devkit_Connectors:DEVKIT_C2000_ROW_B
- removed J3: NAPPE_ADC1, symbol C2000_Devkit_Connectors:NAPPE_ADC1
- removed J4: NAPPE_ADC2, symbol C2000_Devkit_Connectors:NAPPE_ADC2
- removed J5: NAPPE_PWM, symbol C2000_Devkit_Connectors:NAPPE_PWM
- removed J6: NAPPE_GPIO, symbol C2000_Devkit_Connectors:NAPPE_GPIO
- removed J7, J8: ALIM_5V, symbol C2000_Devkit_Connectors:ALIM_5V
- removed J9: ESP32_C6_DEVKITC_1_J1, symbol ESP32_C6_Devkit:ESP32_C6_DEVKITC_1_J1
Other:
- added sheet Connecteurs_Devkit (connecteur_devkit.kicad_sch)
- added sheet Connecteurs_Nappe (connecteurs_nappe.kicad_sch)
- added sheet DC (dc.kicad_sch)
- added sheet Protection_Devkit2 (protection_devkit2.kicad_sch)
- added sheet Protection_Devkit3 (protection_devkit3.kicad_sch)
- added sheet Protections_Devkit (protections_devkit.kicad_sch)
