File: protection_devkit3.kicad_sch (KiCad schematic)
At the start: 9 parts

Commit message: CLB du F28P551 en mini-CPLD : report devkit, 4 trios, nappe logic (decision #20)
- Report sur connecteur_devkit.kicad_sch (symboles + labels reels, lib
  externe incluse) du reseequencement devkit (Iin/Iout/V1/Temp1/Temp2/
  ADC_8-12/I_SHUNT*_CMP/I_SHUNT*_MES deplaces) et des 4 broches neuves
  (Stage1_EN=GPIO9, Stage2_EN=GPIO20, HV_EN=GPIO21, Discharge=GPIO41).
- Corrige un erratum trouve en verifiant : protection_devkit3.kicad_sch
  gardait l'ancien nom nFAULT_MCU apres le renommage du connecteur en
  ~{FAULT_MCU}, coupant silencieusement le trio existant (meme categorie
  de bug que l'erratum ADC-2 de la decision #19).
- 4 nouveaux trios de protection D36-39/R35-38/C55-58, R=10R (signaux
  classes Rapide, decision explicite), pour les 4 sorties neuves.
- Nappe GPIO-2 renommee nappe "logic" (NAPPE_LOGIC, J13) : 9 reserves
  deviennent CLB_Out_1-4/CLB_In_1-5 (noms cosmetiques sur le connecteur
  uniquement, le net electrique reste le vrai nom de signal). 4 sorties
  protegees + 5 entrees tapees sans sacrifice (CAN_RX/CAN_TX, PWM2_B/
  PWM3_B/PWM4_B - deja protegees ailleurs, lues en plus ici).
- netclass_patterns, used_designators, doc/decisions.md #20,
  doc/nappes-shield.md, doc/brochage-devkit.csv mis a jour.

ERC : isolated_pin_label 9->5 (reste les 5 reserves ADC libres, hors
perimetre), pin_not_connected -9 (nappe logic cablee), aucune nouvelle
categorie.
Connections:
- net nFAULT_MCU renamed ~{FAULT_MCU}
Changed lines of the file:
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@@
 		)
 	)
-	(global_label "nFAULT_MCU"
+	(global_label "~{FAULT_MCU}"
 		(shape input)
 		(at 64.33 55.306 180)
@@
 		)
 	)
-	(global_label "nFAULT_MCU"
+	(global_label "~{FAULT_MCU}"
 		(shape input)
 		(at 54.864 47.498 0)
@@
 		)
 	)
-	(global_label "nFAULT_MCU"
+	(global_label "~{FAULT_MCU}"
 		(shape input)
 		(at 50.546 73.152 90)
