File: connecteur_devkit.kicad_sch (KiCad schematic)
At the start: 8 parts, among them J10 OLED_SPI_2x8, J17 DEVKIT_C2000_A, J18 DEVKIT_C2000_B, J7 ESP32_C6_DEVKITC_1_J1, J8 ESP32_C6_DEVKITC_1_J3, U4 ER-OLEDM032-1

Commit message: Resauvegarde session KiCad GUI (placement, empreintes USB-C/STUSB4531, PCB)
Checkpoint avant l'ajout des connecteurs dedies carte HV/Filament -
capture l'etat courant de la session KiCad ouverte (reformattage
eeschema, ajustements d'empreinte sur 632722100213 et STUSB4531QTR,
mises a jour PCB/projet) avant toute edition programmatique.
Other:
- moved on the sheet: J17, J18
