File: usb_pd.kicad_sch (KiCad schematic)
At the start: 24 parts, among them J15 632722100213, J16 CONN_2PIN, Q1 SQJ459EP-T2_GE3, U5 STUSB4531QTR

Commit message: Resauvegarde session KiCad GUI (placement, empreintes USB-C/STUSB4531, PCB)
Checkpoint avant l'ajout des connecteurs dedies carte HV/Filament -
capture l'etat courant de la session KiCad ouverte (reformattage
eeschema, ajustements d'empreinte sur 632722100213 et STUSB4531QTR,
mises a jour PCB/projet) avant toute edition programmatique.
Parts:
- removed D40: ESDA25W, Package_TO_SOT_SMD:SOT-323_SC-70, symbol Power_Parts:ESDA25W
- removed D41, D42: ESDA25P35, Diode_SMD:ST_QFN-2L_1.6x1.0mm, symbol Device:D_TVS
- added D40, D41: Z3SMCxxx, Diode_SMD:D_SMC, symbol Diode:Z3SMCxxx
- added D43: ESDA25W, Package_TO_SOT_SMD:SOT-23-3, symbol Power_Protection:ESDA5V3L
- J15: value 632722100213 -> USBC-PD
Connections:
- net CC1: now also D43.2 (K)
- net CC2: now also D43.1 (K)
- net GND: now also D40.2 (A), D41.2 (A), D43.3 (A)
- net VBUS_IN: now also D40.1 (K)
- net VBUS_OUT: now also D41.1 (K)
- net LED1_A: no longer names the net of LED1.2 (A), R43.2
- net LED2_A: no longer names the net of LED2.2 (A), R44.2
Other:
- title: Alimentation cartes filles - USB-C Power Delivery (STUSB4531QTR, 100W/20V/5A) -> Alimentation USB-C Power Delivery (100W/20V/5A)
- moved on the sheet: C62, C63, C64, C65, J16, LED1, LED2, Q1, R39, R40, R41, R42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
