File: connecteur_ht.kicad_sch (KiCad schematic)
At the start: 16 parts, among them J21 NAPPE_FILAMENT_HT

Commit message: Espace les composants de protection sur connecteur_ht.kicad_sch (anti-chevauchement)
Les 5 trios R+BAT54S+C (Vht/Temp_ht/I_Shunt_ht/I_Shunt_ht_comp/V_bias)
se chevauchaient visuellement (BAT54S empietait sur R et C). Repris au
style defini par l'utilisateur sur le trio Vht : composants en
rotation 90 (horizontal), ~15mm entre les corps, relies par fil+jonction
plutot que par coincidence de label pour les connexions internes locales
au trio (exception documentee au style labels-only, juste pour ce
regroupement physique).

Verifie : check_schematic_labels.py propre, ERC Connecteur_HT toujours
a 0 violation.

Co-Authored-By: Claude Sonnet 5 <noreply@anthropic.com>
Connections:
- net ADC_10_MCU: now also C67.1, R51.2; no longer R51.1
- net ADC_11_MCU: now also C68.1, R52.2; no longer R52.1
- net ADC_12_MCU: now also C70.1, R54.2; no longer R54.1
- net ADC_8_MCU: now also C69.1, R53.2; no longer R53.1
- net ADC_9_MCU: now also C66.1, R50.2; no longer R50.1
- net I_Shunt_ht: now also R52.1; no longer C68.1, R52.2
- net I_Shunt_ht_comp: now also R53.1; no longer C69.1, R53.2
- net Temp_ht: now also R51.1; no longer C67.1, R51.2
- net V_bias: now also R54.1; no longer C70.1, R54.2
- net Vht: now also R50.1; no longer C66.1, R50.2
Other:
- moved on the sheet: C66, D44, R50
